File: right.kicad_pcb (KiCad board)
At the start: 2 copper layers, 150.9 x 130.2 mm, 80 parts, among them J1 AudioJack4, J2 USB_B_Micro, SW1 SW_DIP_x01, SW10 SW_DIP_x01, SW11 SW_DIP_x01, SW12 SW_DIP_x01, SW13 SW_DIP_x01, SW14 SW_DIP_x01, SW15 SW_DIP_x01, SW16 SW_DIP_x01, SW17 SW_DIP_x01, SW18 SW_DIP_x01, SW19 SW_DIP_x01, SW2 SW_DIP_x01, SW20 SW_DIP_x01, SW21 SW_DIP_x01, SW22 SW_DIP_x01, SW23 SW_DIP_x01, SW24 SW_DIP_x01, SW25 SW_DIP_x01, SW26 SW_DIP_x01, SW27 SW_DIP_x01, SW28 SW_DIP_x01, SW29 SW_DIP_x01, SW3 SW_DIP_x01, SW30 SW_Push_Dual, SW4 SW_DIP_x01, SW5 SW_DIP_x01, SW6 SW_DIP_x01, SW7 SW_DIP_x01, SW8 SW_DIP_x01, SW9 SW_DIP_x01, Y1 16MHz

Commit message: Components placed.
Parts:
- moved C1 141.0 mm to (-29.1, 6.06), turned to 180 degrees
- moved C11 135.9 mm to (-30.1, 14.3), turned to 180 degrees
- moved R1 122.7 mm to (-2.56, 6.99)
- moved C6 122.6 mm to (-15.8, 27.6)
- moved C8 117.6 mm to (-24.8, 27.2), turned to 180 degrees
- moved R3 115.7 mm to (-2.60, 20.4)
- moved C2 113.7 mm to (-1.96, 26.5), turned to 270 degrees
- moved C5 113.0 mm to (-8.88, 6.10)
- moved R2 112.9 mm to (-2.60, 18.4)
- moved C7 112.0 mm to (-7.71, 17.3)
- moved C10 110.5 mm to (-7.77, 22.1)
- moved C4 108.9 mm to (-5.87, 26.5), turned to 270 degrees
- moved Y1 108.5 mm to (-18.9, 6.02)
- moved C3 105.6 mm to (1.77, 26.5), turned to 270 degrees
- moved mcu1 103.2 mm to (-19.3, 17.5), turned to 180 degrees
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
Commit message: Layout done.
Parts:
- moved D5 12.8 mm to (-23.6, -6.58), turned to 180 degrees
- moved D27 7.08 mm to (3.57, -4.27), turned to 90 degrees
- moved C8 6.10 mm to (-29.5, 23.2)
- moved C6 1.27 mm to (-15.7, 26.3)
- moved mcu1 1.01 mm to (-19.3, 16.5)
- moved C12 0.97 mm to (-11.1, 25.9)
- moved C3 0.97 mm to (1.29, 25.6)
- moved R3 0.96 mm to (-2.67, 19.5)
- moved R2 0.92 mm to (-2.67, 17.5)
- moved C2 0.90 mm to (-2.26, 25.6)
- moved F1 0.86 mm to (26.3, 1.25)
- moved C4 0.83 mm to (-5.79, 25.6)
- moved C7 0.63 mm to (-7.82, 16.6)
- moved C13 0.62 mm to (-7.81, 14.6)
- moved Y1 0.42 mm to (-19.1, 5.65)
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Routing:
- net /Sheet60738A9D/row0: track 0.00 -> 255.8 mm, vias 0 -> 2
- net /Sheet60738A9D/col0: track 0.00 -> 237.1 mm, vias 0 -> 2
- net /Sheet60738A9D/row3: track 0.00 -> 234.6 mm, vias 0 -> 18
- net /Sheet60738A9D/row1: track 0.00 -> 219.5 mm, vias 0 -> 11
- net /Sheet60738A9D/row4: track 0.00 -> 206.9 mm, vias 0 -> 8
- net /Sheet60738A9D/row2: track 0.00 -> 201.4 mm, vias 0 -> 9
- net /Sheet60738A9D/col5: track 0.00 -> 164.7 mm, vias 0 -> 4
- net /Sheet60738A9D/col2: track 0.00 -> 155.4 mm, vias 0 -> 2
- net /Sheet60738A9D/col3: track 0.00 -> 149.0 mm, vias 0 -> 2
- net /Sheet60738A9D/col1: track 0.00 -> 146.4 mm, vias 0 -> 2
- net /Sheet60738A9D/col4: track 0.00 -> 146.0 mm, vias 0 -> 2
- net UVCC: track 0.00 -> 141.9 mm
- net GND1: track 0.00 -> 68.0 mm, vias 0 -> 27
- net Net-(J1-PadR1): track 0.00 -> 64.9 mm
- net /Sheet60738E4E/USB_FULL1_N: track 0.00 -> 37.4 mm
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- added copper zone on B.Cu, net GND1
Other:
- net class USB_FULL added: clearance 0.2, trace_width 0.5, via_dia 0.8, via_drill 0.4
- net class USB_PWR added: clearance 0.2, trace_width 0.3, via_dia 0.8, via_drill 0.4

Commit message: Minor changes
Parts:
- added REF**: KiCad-Logo_8mm_SilkScreen, Symbol:KiCad-Logo_8mm_SilkScreen, F.Cu at (-83.8, 12.4)
- added REF**: OSHW-Logo2_24.3x20mm_SilkScreen, Symbol:OSHW-Logo2_24.3x20mm_SilkScreen, F.Cu at (-62.9, 14.0)
Other:
- board text added: "Copyright © 2021 Herman Lundkvist Grapto Keyboard, Right PCB v1.0"

Commit message: Fix silkscreen clearance.
Parts:
- moved C10 205.0 mm to (161.2, 138.1)
- moved C8 205.0 mm to (139.6, 139.3)
- moved C9 205.0 mm to (160.1, 126.2)
- moved D2 205.0 mm to (172.2, 81.9)
- moved D27 205.0 mm to (172.6, 111.8)
- moved D3 205.0 mm to (172.2, 62.8)
- moved D4 205.0 mm to (172.2, 43.7)
- moved D5 205.0 mm to (145.4, 109.5)
- moved D6 205.0 mm to (153.1, 97.0)
- moved D7 205.0 mm to (153.1, 77.9)
- moved D8 205.0 mm to (153.1, 58.8)
- moved D9 205.0 mm to (153.1, 39.7)
- moved SW27 205.0 mm to (170.4, 118.2)
- moved SW28 205.0 mm to (190.1, 126.4)
- moved mcu1 205.0 mm to (149.7, 132.6)
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